File: elec/layout/default/veramonitor.kicad_pcb (KiCad board)
At the start: 2 copper layers, 40 x 40 mm, 0 parts

Commit message: great success
Parts:
- added C1: 25V 10uF X5R ±10% 0805 Multilayer Ceramic Capacitors MLCC -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, lib:C0805, F.Cu at (43.4, 126.9)
- added C10: 16V 100nF X7R ±10% 0402 Multilayer Ceramic Capacitors MLCC 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, lib:C0402, F.Cu at (56.9, 144.4)
- added C11: 16V 100nF X7R ±10% 0402 Multilayer Ceramic Capacitors MLCC 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, lib:C0402, F.Cu at (61.9, 144.4)
- added C12: 16V 100nF X7R ±10% 0402 Multilayer Ceramic Capacitors MLCC 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, lib:C0402, F.Cu at (67.0, 144.4)
- added C13: 16V 100nF X7R ±10% 0402 Multilayer Ceramic Capacitors MLCC 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, lib:C0402, F.Cu at (71.9, 144.4)
- added C14: 16V 100nF X7R ±10% 0402 Multilayer Ceramic Capacitors MLCC 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, lib:C0402, F.Cu at (76.9, 144.4)
- added C15: 16V 100nF X7R ±10% 0402 Multilayer Ceramic Capacitors MLCC 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, lib:C0402, F.Cu at (81.8, 144.4)
- added C16: 16V 100nF X7R ±10% 0402 Multilayer Ceramic Capacitors MLCC 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, lib:C0402, F.Cu at (86.7, 144.4)
- added C17: 16V 100nF X7R ±10% 0402 Multilayer Ceramic Capacitors MLCC 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, lib:C0402, F.Cu at (91.6, 144.4)
- added C18: 16V 100nF X7R ±10% 0402 Multilayer Ceramic Capacitors MLCC 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, lib:C0402, F.Cu at (96.6, 144.3)
- added C19: 16V 100nF X7R ±10% 0402 Multilayer Ceramic Capacitors MLCC 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, lib:C0402, F.Cu at (101.6, 144.3)
- added C2: 25V 10uF X5R ±10% 0805 Multilayer Ceramic Capacitors MLCC -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, lib:C0805, F.Cu at (46.2, 124.7)
- added C20: 16V 100nF X7R ±10% 0402 Multilayer Ceramic Capacitors MLCC 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, lib:C0402, F.Cu at (106.6, 144.3)
- added C21: 16V 100nF X7R ±10% 0402 Multilayer Ceramic Capacitors MLCC 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, lib:C0402, F.Cu at (111.6, 144.3)
- added C22: 16V 100nF X7R ±10% 0402 Multilayer Ceramic Capacitors MLCC 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, lib:C0402, F.Cu at (116.7, 144.3)
- added C23: 16V 100nF X7R ±10% 0402 Multilayer Ceramic Capacitors MLCC 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, lib:C0402, F.Cu at (121.6, 144.3)
- added C24: 16V 100nF X7R ±10% 0402 Multilayer Ceramic Capacitors MLCC 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, lib:C0402, F.Cu at (126.7, 144.3)
- added C25: 16V 100nF X7R ±10% 0402 Multilayer Ceramic Capacitors MLCC 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, lib:C0402, F.Cu at (131.5, 144.3)
- added C3: 16V 100nF X7R ±10% 0402 Multilayer Ceramic Capacitors MLCC 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, lib:C0402, F.Cu at (51.8, 122.0)
- added C4: 25V 10uF X5R ±10% 0805 Multilayer Ceramic Capacitors MLCC -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, lib:C0805, F.Cu at (50.1, 121.3)
- added C5: 25V 10uF X5R ±10% 0805 Multilayer Ceramic Capacitors MLCC -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, lib:C0805, F.Cu at (48.0, 121.3)
- added C6: 16V 100nF X7R ±10% 0402 Multilayer Ceramic Capacitors MLCC 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, lib:C0402, F.Cu at (37.0, 144.5)
- added C7: 16V 100nF X7R ±10% 0402 Multilayer Ceramic Capacitors MLCC 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, lib:C0402, F.Cu at (41.9, 144.5)
- added C8: 16V 100nF X7R ±10% 0402 Multilayer Ceramic Capacitors MLCC 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, lib:C0402, F.Cu at (46.9, 144.4)
- added C9: 16V 100nF X7R ±10% 0402 Multilayer Ceramic Capacitors MLCC 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, lib:C0402, F.Cu at (51.9, 144.4)
- added J1: ?, lib:CONN-SMD_4P-P1.00_SM04B-SRSS-TB-LF-SN, F.Cu at (37.5, 124.7)
- added R1: 62.5mW Thick Film Resistors 50V ±100ppm/℃ ±1% 5.1kΩ 0402 Ch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, lib:R0402, F.Cu at (42.8, 132.4)
- added R2: 62.5mW Thick Film Resistors 50V ±100ppm/℃ ±1% 5.1kΩ 0402 Ch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, lib:R0402, F.Cu at (42.8, 135.5)
- added R3: 62.5mW Thick Film Resistors 50V ±100ppm/℃ ±1% 10kΩ 0402 Chi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, lib:R0402, F.Cu at (51.8, 123.7)
- added U1: ?, lib:TAG-CONNECT_TC2050-IDC, F.Cu at (76.8, 129.5)
- added U10: ?, lib:LED-SMD_4P-L2.0-W2.0-BR, F.Cu at (51.7, 142.6)
- added U11: ?, lib:LED-SMD_4P-L2.0-W2.0-BR, F.Cu at (56.7, 142.6)
- added U12: ?, lib:LED-SMD_4P-L2.0-W2.0-BR, F.Cu at (61.7, 142.6)
- added U13: ?, lib:LED-SMD_4P-L2.0-W2.0-BR, F.Cu at (66.7, 142.6)
- added U14: ?, lib:LED-SMD_4P-L2.0-W2.0-BR, F.Cu at (71.7, 142.6)
- added U15: ?, lib:LED-SMD_4P-L2.0-W2.0-BR, F.Cu at (76.7, 142.6)
- added U16: ?, lib:LED-SMD_4P-L2.0-W2.0-BR, F.Cu at (81.7, 142.6)
- added U17: ?, lib:LED-SMD_4P-L2.0-W2.0-BR, F.Cu at (86.5, 142.6)
- added U18: ?, lib:LED-SMD_4P-L2.0-W2.0-BR, F.Cu at (91.5, 142.6)
- added U19: ?, lib:LED-SMD_4P-L2.0-W2.0-BR, F.Cu at (96.5, 142.6)
- added U2: ?, lib:USB-C-SMD_KH-TYPE-C-16P, F.Cu at (38.5, 133.9)
- added U20: ?, lib:LED-SMD_4P-L2.0-W2.0-BR, F.Cu at (101.5, 142.6)
- added U21: ?, lib:LED-SMD_4P-L2.0-W2.0-BR, F.Cu at (106.5, 142.6)
- added U22: ?, lib:LED-SMD_4P-L2.0-W2.0-BR, F.Cu at (111.5, 142.6)
- added U23: ?, lib:LED-SMD_4P-L2.0-W2.0-BR, F.Cu at (116.5, 142.6)
- added U24: ?, lib:LED-SMD_4P-L2.0-W2.0-BR, F.Cu at (121.5, 142.6)
- added U25: ?, lib:LED-SMD_4P-L2.0-W2.0-BR, F.Cu at (126.5, 142.6)
- added U26: ?, lib:LED-SMD_4P-L2.0-W2.0-BR, F.Cu at (131.5, 142.6)
- added U3: ?, lib:MIC-SMD_5P_L3.5-W2.7-P0.82_SPH0641LU4H-1, F.Cu at (48.1, 137.4)
- added U4: ?, lib:SOT-223-3_L6.5-W3.4-P2.30-LS7.0-BR, F.Cu at (47.5, 130.2)
- added U5: ?, lib:WIRELM-SMD_ESP32-S3-WROOM-1, F.Cu at (62.5, 130.1)
- added U6: ?, lib:KEY-SMD_4P-L4.2-W3.2-P2.20-LS4.6, F.Cu at (44.0, 121.2)
- added U7: ?, lib:LED-SMD_4P-L2.0-W2.0-BR, F.Cu at (36.7, 142.6)
- added U8: ?, lib:LED-SMD_4P-L2.0-W2.0-BR, F.Cu at (41.7, 142.6)
- added U9: ?, lib:LED-SMD_4P-L2.0-W2.0-BR, F.Cu at (46.7, 142.6)
Routing:
- net gnd: track 0.00 -> 314.7 mm, vias 0 -> 40
- net vcc: track 0.00 -> 176.0 mm, vias 0 -> 20
- net led_data: track 0.00 -> 28.9 mm
- net pdm_clk: track 0.00 -> 20.6 mm, vias 0 -> 2
- net vcc-1: track 0.00 -> 17.5 mm
- net pdm_data: track 0.00 -> 16.0 mm, vias 0 -> 2
- net dp: track 0.00 -> 14.5 mm
- net dm: track 0.00 -> 14.2 mm
- net pdm_sel: track 0.00 -> 11.0 mm, vias 0 -> 2
- net tdo: track 0.00 -> 9.05 mm, vias 0 -> 2
- net tdi: track 0.00 -> 8.60 mm, vias 0 -> 2
- net tms: track 0.00 -> 5.12 mm
- net tck: track 0.00 -> 5.05 mm
- net ledrow2.led8.ic-vcc: track 0.00 -> 4.24 mm
- net ledrow2.led5.ic-vcc: track 0.00 -> 4.24 mm
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Other:
- board outline removed
- board text removed: "{{GITHASH}}"
