File: elec/layout/default/veramonitor.kicad_pcb (KiCad board)
At the start: 2 copper layers, 105.2 x 61.6 mm, 48 parts, among them J1 ?, U1 ?, U10 ?, U11 ?, U12 ?, U13 ?, U14 ?, U15 ?, U16 ?, U17 ?, U18 ?, U19 ?, U2 ?, U20 ?, U21 ?, U22 ?, U3 ?, U4 ?, U5 ?, U6 ?, U7 ?, U8 ?, U9 ?

Commit message: :woozy:
Parts:
- C1: value 50V 10nF X7R ±10% 0402 Multilayer Ceramic Capacitors MLCC - SMD/SMT ROHS -> (none); footprint lib:C0402 -> atopile:C_0402_1005Metric
- C10, C11, C12, C13, C14, C4, C8, C9: value 16V 100nF X7R ±10% 0402 Multilayer Ceramic Capacitors MLCC - SMD/SMT ROHS -> 100nF ±10% 16V X7R; footprint lib:C0402 -> atopile:C0402-b3ef17
- C2, C3, C5, C6: value 25V 10uF X5R ±10% 0805 Multilayer Ceramic Capacitors MLCC - SMD/SMT ROHS -> 10µF ±10% 25V X5R; footprint lib:C0805 -> atopile:C0805-3b2e55
- C7: value 6.3V 10uF X5R ±20% 0402 Multilayer Ceramic Capacitors MLCC - SMD/SMT ROHS -> 10µF ±20% 6.3V X5R; footprint lib:C0402 -> atopile:C0402-b3ef17
- J1, U1, U10, U11, U12, U13, U14, U15, U16, U17, U18, U19, U2, U20, U21, U22, U3, U4, U5, U6, U7, U8, U9: value ? -> (none)
- R1, R2: value 62.5mW Thick Film Resistors 50V ±100ppm/℃ ±1% 4.7kΩ 0402 Chip Resistor - Surface Mount ROHS -> 4.7kΩ ±1% 62.5mW; footprint lib:R0402 -> atopile:R0402-56259e
- R10, R5, R6, R7, R8, R9: value 50mW Thick Film Resistors 25V ±1% ±200ppm/℃ 10kΩ 0201 Chip Resistor - Surface Mount ROHS -> 10kΩ ±1% 62.5mW; footprint lib:R0201 -> atopile:R0402-56259e
- R11, R3, R4: value 62.5mW Thick Film Resistors 50V ±100ppm/℃ ±1% 10kΩ 0402 Chip Resistor - Surface Mount ROHS -> 10kΩ ±1% 62.5mW; footprint lib:R0402 -> atopile:R0402-56259e
Connections:
- net backlighten renamed BL
- net bclk renamed BCLK
- net cc1 renamed CC1
- net cc2 renamed B5
- net dc renamed DC
- net din renamed DIN-1
- net dummy renamed DUMMY
- net en renamed in-1
- net gain_slot renamed GAIN_SLOT
- net io14 renamed KEY-1
- net io16 renamed DIN
- net io21 renamed KEY-3
- net io35 renamed KEY-4
- net io45 renamed KEY
- net io47 renamed KEY-2
- net io48 renamed KEY-5
- net jtag_connector-reset renamed reset-1
- net lrclk renamed LRCLK
- net micro.ic-reset renamed reset
- net micro.ic-vcc renamed in
- net mosi renamed DIN-2
- net n_period_c_period renamed N_period_C_period
- net outn renamed OUTN
- net outp renamed OUTP
- net pdm_data renamed DATA
- net pdm_sel renamed SELECT
- net rxd0 renamed rx
- net scl renamed line
- net sd_mode_hash renamed SD_MODE_hash
- net sda renamed line-1
- net sub1 renamed SUB1
- net sub2 renamed B8
- net sw1-dout renamed io-1
- net sw3-dout renamed io
- net sw4-dout renamed io-2
- net sw6-dout renamed DOUT
- net txd0 renamed tx
- C1 pad 1: vcc-1 -> hv-1
- C10 pad 1: vcc-1 -> hv-1
- C11 pad 1: vcc-1 -> hv-1
- C12 pad 1: vcc-1 -> hv-1
- C13 pad 1: vcc-1 -> hv-1
- C14 pad 1: vcc-1 -> hv-1
- C2 pad 1: vcc -> hv
- C3 pad 1: vcc-1 -> hv-1
- C4 pad 1: vcc-1 -> hv-1
- C5 pad 1: vcc-1 -> hv-1
- C6 pad 1: vcc-1 -> hv-1
- C7 pad 1: vcc-1 -> hv-1
- C8 pad 1: vcc-1 -> hv-1
- C9 pad 1: vcc-1 -> hv-1
- J1 pad 2: vcc-1 -> hv-1
- R10 pad 1: vcc-1 -> hv-1
- R11 pad 1: vcc-1 -> hv-1
- R3 pad 1: vcc-1 -> hv-1
- R4 pad 1: vcc-1 -> hv-1
- R5 pad 1: vcc-1 -> hv-1
- R6 pad 1: vcc-1 -> hv-1
- R7 pad 1: vcc-1 -> hv-1
- R8 pad 1: vcc-1 -> hv-1
- R9 pad 1: vcc-1 -> hv-1
- U1 pad 1: vcc -> hv
- U11 pad 1: vcc-1 -> hv-1
- U11 pad 2: sw2-dout -> vcc
- U13 pad 1: vcc-1 -> hv-1
- U13 pad 4: sw2-dout -> vcc
- U15 pad 1: vcc-1 -> hv-1
- U17 pad 1: vcc-1 -> hv-1
- U17 pad 2: sw5-dout -> vcc-1
- U19 pad 1: vcc-1 -> hv-1
- U19 pad 4: sw5-dout -> vcc-1
- U2 pad A4: vcc -> hv
- U2 pad A9: vcc -> hv
- U2 pad B4: vcc -> hv
- U2 pad B9: vcc -> hv
- U3 pad 5: vcc-1 -> hv-1
- U4 pad 2: vcc-1 -> hv-1
- U4 pad 3: vcc -> hv
- U4 pad 4: vcc-1 -> hv-1
- U5 pad 2: vcc-1 -> hv-1
- U7 pad 1: vcc -> hv
- U8 pad 7: vcc-1 -> hv-1
- U8 pad 8: vcc-1 -> hv-1
- U9 pad 1: vcc-1 -> hv-1
Routing:
- net hv-1: track 0.00 -> 356.5 mm, vias 0 -> 11
- net vcc-1: track 356.5 -> 24.5 mm, vias 11 -> 2
- net hv: track 0.00 -> 103.1 mm, vias 0 -> 4
- net vcc: track 103.1 -> 16.9 mm, vias 4 -> 2
- net sw5-dout: track 24.5 -> 0.00 mm, vias 2 -> 0
- net sw2-dout: track 16.9 -> 0.00 mm, vias 2 -> 0
Other:
- board text added: "{{GITHASH}}"

Commit message: editing layout
Parts:
- moved U5 6.09 mm to (56.6, 78.8)
- moved R11 5.90 mm to (65.7, 67.8)
- moved U1 5.90 mm to (53.6, 64.8)
- moved U22 5.90 mm to (62.1, 66.0)
- moved U7 5.10 mm to (73.1, 82.2)
- moved C14 3.27 mm to (136.9, 82.0)
- moved R10 3.27 mm to (128.7, 74.4)
- moved U19 3.27 mm to (137.0, 78.4)
- moved U20 3.27 mm to (136.4, 69.6)
- moved R9 2.87 mm to (128.6, 94.1)
- moved C13 2.87 mm to (137.1, 101.2)
- moved U17 2.87 mm to (137.2, 97.6)
- moved U18 2.87 mm to (136.4, 88.8)
- moved U16 2.73 mm to (136.4, 107.7)
- moved R8 2.73 mm to (128.7, 111.7)
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Routing:
- net KEY: track 93.0 -> 9.96 mm
- net KEY-2: track 76.3 -> 10.1 mm
- net KEY-5: track 93.8 -> 35.0 mm
- net KEY-1: track 58.1 -> 8.98 mm
- net KEY-3: track 67.2 -> 24.0 mm
- net hv: track 103.1 -> 67.7 mm
- net io-2: track 24.6 -> 0.00 mm
- net io: track 17.5 -> 42.1 mm
- net vcc-1: track 24.5 -> 0.00 mm
- net line: track 22.3 -> 0.00 mm
- net DIN: track 48.9 -> 27.9 mm, vias 2 -> 1
- net line-1: track 20.2 -> 0.14 mm
- net hv-1: track 356.5 -> 336.7 mm
- net pdm_clk: track 15.9 -> 3.76 mm
- net DATA: track 14.4 -> 2.39 mm
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Other:
- board size 105.2 x 61.6 mm -> 107.7 x 61.6 mm
- board text added: "izzymonitor :3"
- board text removed: "izzymonitor :3 December 2024"
