File: elec/src/esp32-s3/elec/layout/default/esp32-s3.kicad_pcb (KiCad board)
At the start: 2 copper layers, 6 parts

Commit message: great success
Parts:
- moved C1 80.9 mm to (39.6, 131.8)
- moved C3 80.8 mm to (35.8, 131.1)
- moved C2 80.7 mm to (37.9, 131.1)
- moved U1 80.5 mm to (50.4, 139.8)
- moved R1 79.9 mm to (39.6, 133.5), turned to 0 degrees
- moved U2 74.6 mm to (37.5, 126.4), turned to 180 degrees
Routing:
- net en: track 8.40 -> 0.00 mm
- net vcc: track 7.15 -> 0.00 mm
- net ic-gnd: track 5.54 -> 0.00 mm
